File: eagle/i2cstump-usbc.brd (EAGLE design)
At the start: 25.9 x 18.8 mm, 22 parts, among them IC1 ATTINY85, IC2 MCP1703CB, J1 I2C-5V, J2 I2C-3V3, Q1 220mA/50V/3.5Ω, Q2 220mA/50V/3.5Ω

Commit message: Correct value of R7 (390R)
Parts:
- R7: value 2k2 -> 390R
Changed lines of the file:
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@@
 <?xml version="1.0" encoding="utf-8"?>
 <!DOCTYPE eagle SYSTEM "eagle.dtd">
-<eagle version="9.2.2">
+<eagle version="9.4.1">
 <drawing>
 <settings>
@@
 <attribute name="VALUE" x="10.16" y="7.366" size="0.6096" layer="27" font="vector" ratio="20" rot="R180" align="top-center"/>
 </element>
-<element name="R7" library="SparkFun-Resistors" library_urn="urn:adsk.eagle:library:532" package="0603" package3d_urn="urn:adsk.eagle:package:39650/1" value="2k2" x="7.112" y="3.302" smashed="yes">
+<element name="R7" library="SparkFun-Resistors" library_urn="urn:adsk.eagle:library:532" package="0603" package3d_urn="urn:adsk.eagle:package:39650/1" value="390R" x="7.112" y="3.302" smashed="yes">
 <attribute name="NAME" x="7.493" y="4.064" size="0.6096" layer="25" font="vector" ratio="20" align="bottom-center"/>
 <attribute name="PROD_ID" value=" " x="7.112" y="3.302" size="1.778" layer="27" display="off"/>

Commit message: Change red PWR led to be 1k resistor so it's not as bright. Conversely, lower green ACT led to 330R so it's a bit brighter
Parts:
- R3: value 390R -> 330R
- R7: value 390R -> 1k
Changed lines of the file:
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@@
 <?xml version="1.0" encoding="utf-8"?>
 <!DOCTYPE eagle SYSTEM "eagle.dtd">
-<eagle version="9.4.1">
+<eagle version="9.2.2">
 <drawing>
 <settings>
@@
 <attribute name="VALUE" x="3.048" y="1.905" size="0.6096" layer="27" font="vector" ratio="20" rot="R180" align="top-center"/>
 </element>
-<element name="R3" library="SparkFun-Resistors" library_urn="urn:adsk.eagle:library:532" package="0603" package3d_urn="urn:adsk.eagle:package:39650/1" value="390R" x="7.112" y="1.27" smashed="yes">
+<element name="R3" library="SparkFun-Resistors" library_urn="urn:adsk.eagle:library:532" package="0603" package3d_urn="urn:adsk.eagle:package:39650/1" value="330R" x="7.112" y="1.27" smashed="yes">
 <attribute name="NAME" x="7.493" y="1.905" size="0.6096" layer="25" font="vector" ratio="20" align="bottom-center"/>
 <attribute name="PROD_ID" value=" " x="7.112" y="1.27" size="1.778" layer="27" display="off"/>
@@
 <attribute name="VALUE" x="10.16" y="7.366" size="0.6096" layer="27" font="vector" ratio="20" rot="R180" align="top-center"/>
 </element>
-<element name="R7" library="SparkFun-Resistors" library_urn="urn:adsk.eagle:library:532" package="0603" package3d_urn="urn:adsk.eagle:package:39650/1" value="390R" x="7.112" y="3.302" smashed="yes">
+<element name="R7" library="SparkFun-Resistors" library_urn="urn:adsk.eagle:library:532" package="0603" package3d_urn="urn:adsk.eagle:package:39650/1" value="1k" x="7.112" y="3.302" smashed="yes">
 <attribute name="NAME" x="7.493" y="4.064" size="0.6096" layer="25" font="vector" ratio="20" align="bottom-center"/>
 <attribute name="PROD_ID" value=" " x="7.112" y="3.302" size="1.778" layer="27" display="off"/>
